File: ESP-Mailbox-rounded.kicad_pcb (KiCad board)
At the start: 2 copper layers, 79 x 25 mm, 21 parts, among them J1 FTDI, J2 EXTRESET, SW1 RESET, SW2 FLASH, U1 BRCL3130MC, U2 ESP-M2, U3 ME6811

Commit message: updates
Routing:
- net +3.3V: track 69.9 -> 72.8 mm
- net GND: vias 21 -> 23
Other:
- board text added: "+"
- board text added: "-"
