File: ESP-Mailbox.kicad_sch (KiCad schematic)
At the start: 21 parts, among them J1 FTDI, J2 EXTRESET, SW1 RESET, SW2 FLASH, U1 BRCL3130MC, U2 ESP-M2, U3 ME6811

Commit message: updates
Parts:
- U3: value ME6811 -> ME6209
Changed lines of the file:
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@@
     (in_bom yes) (on_board yes) (fields_autoplaced)
     (property "Reference" "U3" (id 0) (at 93.98 29.21 0))
-    (property "Value" "ME6811" (id 1) (at 93.98 31.75 0))
+    (property "Value" "ME6209" (id 1) (at 93.98 31.75 0))
     (property "Footprint" "Package_TO_SOT_SMD:SOT-23_Handsoldering" (id 2) (at 93.98 31.115 0)
       (effects (font (size 1.27 1.27)) hide)
@@
     )
     (path "/2e766d16-9d8f-4bbf-b0e2-ae85e471c358"
-      (reference "U3") (unit 1) (value "ME6811") (footprint "Package_TO_SOT_SMD:SOT-23_Handsoldering")
-    )
-  )
+      (reference "U3") (unit 1) (value "ME6209") (footprint "Package_TO_SOT_SMD:SOT-23_Handsoldering")
+    )
+  )
